File: docs/kicad/node.kicad_sch (KiCad schematic)
At the start: 9 parts, among them U1 ESP32-DevKitC, U2 ESP32-DevKitC, U3 ESP32-DevKitC, U4 ESP32-DevKitC

Commit message: update kicad model
Parts:
- removed JP1, JP2, JP7, JP8, JP9: Jumper_2_Open, Connector_PinSocket_1.00mm:PinSocket_1x02_P1.00mm_Vertical, symbol Jumper:Jumper_2_Open
- removed U1, U2, U3, U4: ESP32-DevKitC, PCM_Espressif:ESP32-DevKitC, symbol PCM_Espressif:ESP32-DevKitC
Other:
- added sheet ap (ap.kicad_sch)
- added sheet main (main.kicad_sch)
- note removed: "By-pass AP"
