File: docs/kicad/node.kicad_pcb (KiCad board)
At the start: 2 copper layers, 181.1 x 116.5 mm, 8 parts, among them J10 Conn_01x04_Pin, J11 Conn_01x04_Pin, J9 Conn_01x08, U1 ESP32-DevKitC, U2 ESP32-DevKitC, U3 ESP32-DevKitC, U4 ESP32-DevKitC, U5 ESP32-DevKitC

Commit message: resolved all errors
Parts:
- moved J10 44.5 mm to (95.0, 76.0), turned to 0 degrees
- moved J11 12.8 mm to (122.0, 130.0)
- moved U1 9.04 mm to (54.0, 131.0)
- moved U4 8.83 mm to (131.0, 98.7)
- moved U3 6.35 mm to (99.0, 22.0)
- moved U2 5.58 mm to (21.3, 53.0)
Routing:
- net /main/B4_CS: track 45.4 -> 10.7 mm
- net /main/B4_SCLK: track 41.8 -> 10.7 mm
- net GND: track 179.7 -> 203.4 mm
- net /main/B5_MOSI: track 45.4 -> 32.5 mm
- net /main/B4_MOSI: track 31.9 -> 19.5 mm
- net /main/B5_SCLK: track 57.2 -> 46.0 mm
- net /main/B5_CS: track 52.8 -> 42.1 mm
- net /main/B1_MOSI: track 39.9 -> 44.8 mm
- net /main/B1_SCLK: track 59.5 -> 63.8 mm
- net /main/B1_CS: track 32.4 -> 36.8 mm
- net /main/B3_MOSI: track 39.7 -> 43.0 mm
- net /main/B2_MOSI: track 40.0 -> 42.7 mm
- net /main/B3_CS: track 32.2 -> 34.9 mm
- net /main/B3_SCLK: track 59.3 -> 62.0 mm
- net /main/VCC: track 310.8 -> 313.2 mm
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Other:
- board size 181.1 x 116.5 mm -> 179.6 x 125 mm

Commit message: nit
Parts:
- moved J10 41.9 mm to (122.0, 108.0), turned to -90 degrees
Routing:
- net /main/B4_CS: track 10.7 -> 39.1 mm
- net /main/B4_SCLK: track 10.7 -> 35.5 mm
- net GND: track 203.4 -> 182.2 mm
- net /main/B4_MOSI: track 19.5 -> 16.5 mm
Changed lines of the file:
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@@
 	(footprint "Connector_PinSocket_2.54mm:PinSocket_1x04_P2.54mm_Vertical"
 		(layer "F.Cu")
-		(at 95 76)
+		(at 122 108 -90)
 		(descr "Through hole straight socket strip, 1x04, 2.54mm pitch, single row (from Kicad 4.0.7), script generated")
 		(tags "Through hole socket strip THT 1x04 2.54mm single row")
 		(property "Reference" "J10"
-			(at 0 -2.77 360)
+			(at 0 -2.77 90)
 			(layer "F.SilkS")
 			(effects
@@
 		)
 		(property "Value" "Conn_01x04_Pin"
-			(at 0 10.39 360)
+			(at 0 10.39 90)
 			(layer "F.Fab")
 			(effects
@@
 		)
 		(property "Footprint" "Connector_PinSocket_2.54mm:PinSocket_1x04_P2.54mm_Vertical"
-			(at 0 0 0)
+			(at 0 0 -90)
 			(unlocked yes)
 			(layer "F.Fab")
@@
 		)
 		(property "Datasheet" ""
-			(at 0 0 0)
+			(at 0 0 -90)
 			(unlocked yes)
 			(layer "F.Fab")
@@
 		)
 		(property "Description" "Generic connector, single row, 01x04, script generated"
-			(at 0 0 0)
+			(at 0 0 -90)
 			(unlocked yes)
 			(layer "F.Fab")
@@
 		(attr through_hole)
 		(fp_line
+			(start -1.33 8.95)
+			(end 1.33 8.95)
+			(stroke
+				(width 0.12)
+				(type solid)
+			)
+			(layer "F.SilkS")
+		)
+		(fp_line
 			(start -1.33 1.27)
 			(end -1.33 8.95)
@@
 		)
 		(fp_line
-			(start -1.33 8.95)
+			(start 1.33 1.27)
 			(end 1.33 8.95)
 			(stroke
@@
 		)
 		(fp_line
-			(start 1.33 1.27)
-			(end 1.33 8.95)
-			(stroke
-				(width 0.12)
-				(type solid)
-			)
-			(layer "F.SilkS")
-		)
-		(fp_line
-			(start -1.8 -1.8)
-			(end 1.75 -1.8)
+			(start -1.8 9.4)
+			(end -1.8 -1.8)
 			(stroke
 				(width 0.05)
@@
 		)
 		(fp_line
-			(start -1.8 9.4)
-			(end -1.8 -1.8)
+			(start 1.75 9.4)
+			(end -1.8 9.4)
 			(stroke
 				(width 0.05)
@@
 		)
 		(fp_line
-			(start 1.75 -1.8)
-			(end 1.75 9.4)
+			(start -1.8 -1.8)
+			(end 1.75 -1.8)
 			(stroke
 				(width 0.05)
@@
 		)
 		(fp_line
-			(start 1.75 9.4)
-			(end -1.8 9.4)
+			(start 1.75 -1.8)
+			(end 1.75 9.4)
 			(stroke
 				(width 0.05)
@@
 		)
 		(fp_line
-			(start -1.27 -1.27)
-			(end 0.635 -1.27)
+			(start -1.27 8.89)
+			(end -1.27 -1.27)
 			(stroke
 				(width 0.1)
@@
 		)
 		(fp_line
-			(start -1.27 8.89)
-			(end -1.27 -1.27)
+			(start 1.27 8.89)
+			(end -1.27 8.89)
 			(stroke
 				(width 0.1)
@@
 		)
 		(fp_line
-			(start 0.635 -1.27)
-			(end 1.27 -0.635)
+			(start 1.27 -0.635)
+			(end 1.27 8.89)
 			(stroke
 				(width 0.1)
@@
 		)
 		(fp_line
-			(start 1.27 -0.635)
-			(end 1.27 8.89)
+			(start -1.27 -1.27)
+			(end 0.635 -1.27)
 			(stroke
 				(width 0.1)
@@
 		)
 		(fp_line
-			(start 1.27 8.89)
-			(end -1.27 8.89)
+			(start 0.635 -1.27)
+			(end 1.27 -0.635)
 			(stroke
 				(width 0.1)
@@
 		)
 		(fp_text user "${REFERENCE}"
-			(at 0 3.81 90)
+			(at 0 3.81 360)
 			(layer "F.Fab")
 			(effects
@@
 		)
 		(pad "1" thru_hole rect
-			(at 0 0)
+			(at 0 0 270)
 			(size 1.7 1.7)
 			(drill 1)
@@
 		)
 		(pad "2" thru_hole oval
-			(at 0 2.54)
+			(at 0 2.54 270)
 			(size 1.7 1.7)
 			(drill 1)
@@
 		)
 		(pad "3" thru_hole oval
-			(at 0 5.08)
+			(at 0 5.08 270)
 			(size 1.7 1.7)
 			(drill 1)
@@
 		)
 		(pad "4" thru_hole oval
-			(at 0 7.62)
+			(at 0 7.62 270)
 			(size 1.7 1.7)
 			(drill 1)
@@
 	)
 	(gr_text "AP_CS\nAP_SCLK\nAP_MOSI\nVCC"
-		(at 113 128 270)
+		(at 126 132 270)
 		(layer "F.Cu")
 		(effects
@@
 	)
 	(gr_text "EAST_CS\nEAST_SCLK\nEAST_MOSI\nGND"
-		(at 93 85 0)
+		(at 126 106 270)
 		(layer "F.Cu")
 		(effects
@@
 				(bold yes)
 			)
-			(justify right bottom)
+			(justify left bottom)
 		)
 	)
@@
 	)
 	(segment
+		(start 105.6 99.22)
+		(end 105.6 98.72)
+		(width 0.8)
+		(layer "B.Cu")
+		(net 1)
+	)
+	(segment
 		(start 48.3 56.48)
 		(end 48.3 54.6)
@@
 	)
 	(segment
-		(start 49 63.4)
-		(end 46.7 65.7)
+		(start 114.38 108)
+		(end 105.6 99.22)
 		(width 0.8)
 		(layer "B.Cu")
@@
 	)
 	(segment
-		(start 61.68 103)
-		(end 66.64 103)
+		(start 49 63.4)
+		(end 46.7 65.7)
 		(width 0.8)
 		(layer "B.Cu")
@@
 	)
 	(segment
-		(start 105.6 98.72)
-		(end 108 96.32)
+		(start 61.68 103)
+		(end 66.64 103)
 		(width 0.8)
 		(layer "B.Cu")
@@
 	)
 	(segment
-		(start 95 83.62)
-		(end 95 88.12)
-		(width 0.8)
-		(layer "B.Cu")
-		(net 1)
-	)
-	(segment
-		(start 95 88.12)
-		(end 105.6 98.72)
-		(width 0.8)
-		(layer "B.Cu")
-		(net 1)
-	)
-	(segment
 		(start 111.4 47.4)
 		(end 99.02 47.4)
@@
 	)
 	(segment
-		(start 108 96.32)
-		(end 108 88.42)
-		(width 0.8)
-		(layer "B.Cu")
-		(net 1)
-	)
-	(segment
 		(start 21.3 86.02)
 		(end 23.16 86.02)
@@
 	)
 	(segment
-		(start 108 88.42)
-		(end 105.6 86.02)
-		(width 0.8)
-		(layer "B.Cu")
-		(net 1)
-	)
-	(segment
 		(start 21.3 104.3)
 		(end 52 135)
@@
 	)
 	(segment
-		(start 95 76)
-		(end 105.46 76)
+		(start 122 92.26)
+		(end 105.6 75.86)
+		(width 0.8)
+		(layer "B.Cu")
+		(net 3)
+	)
+	(segment
+		(start 122 108)
+		(end 122 92.26)
 		(width 0.8)
 		(layer "B.Cu")
@@
 	)
 	(segment
-		(start 95 78.54)
-		(end 105.46 78.54)
+		(start 119.46 92.26)
+		(end 105.6 78.4)
 		(width 0.8)
 		(layer "B.Cu")
@@
 	)
 	(segment
-		(start 95 81.08)
-		(end 103 89.08)
+		(start 119.46 108)
+		(end 119.46 92.26)
 		(width 0.8)
 		(layer "B.Cu")
-		(net 7)
+		(net 6)
 	)
 	(segment
-		(start 103 89.08)
-		(end 103 93.58)
+		(start 116.92 107.5)
+		(end 105.6 96.18)
 		(width 0.8)
 		(layer "B.Cu")
@@
 	)
 	(segment
-		(start 103 93.58)
-		(end 105.6 96.18)
+		(start 116.92 108)
+		(end 116.92 107.5)
 		(width 0.8)
 		(layer "B.Cu")
